Commit message: Version bump & small fixes
- bumped to 1.7.0
- fixed directory of hexapod meshes
- fixed horizon of hexapodbullet environment

File: mushroom_rl/environments/pybullet_envs/data/hexapod/hexapod.urdf (robot description, URDF)
Before this commit: robot iiwa, 38 links, 37 joints
Links:
- link hexapod/body: geometry collision mesh filename=meshes/collision/base.stl; visual mesh filename=meshes/visual/base.stl
- link hexapod/leg_0/link_0: geometry collision mesh filename=meshes/collision/leg_0_left.stl; visual mesh filename=meshes/visual/leg_0_left.stl
- link hexapod/leg_0/link_1: geometry collision mesh filename=meshes/collision/leg_1.stl; visual mesh filename=meshes/visual/leg_1.stl
- link hexapod/leg_0/link_2: geometry collision mesh filename=meshes/collision/leg_2_left.stl; visual mesh filename=meshes/visual/leg_2_left.stl
- link hexapod/leg_0/motor_0: geometry collision mesh filename=meshes/collision/motor.stl; visual mesh filename=meshes/visual/motor.stl
- link hexapod/leg_0/motor_1: geometry collision mesh filename=meshes/collision/motor.stl; visual mesh filename=meshes/visual/motor.stl
- link hexapod/leg_0/motor_2: geometry collision mesh filename=meshes/collision/motor.stl; visual mesh filename=meshes/visual/motor.stl
- link hexapod/leg_1/link_0: geometry collision mesh filename=meshes/collision/leg_0_right.stl; visual mesh filename=meshes/visual/leg_0_right.stl
- link hexapod/leg_1/link_1: geometry collision mesh filename=meshes/collision/leg_1.stl; visual mesh filename=meshes/visual/leg_1.stl
- link hexapod/leg_1/link_2: geometry collision mesh filename=meshes/collision/leg_2_right.stl; visual mesh filename=meshes/visual/leg_2_right.stl
- link hexapod/leg_1/motor_0: geometry collision mesh filename=meshes/collision/motor.stl; visual mesh filename=meshes/visual/motor.stl
- link hexapod/leg_1/motor_1: geometry collision mesh filename=meshes/collision/motor.stl; visual mesh filename=meshes/visual/motor.stl
- link hexapod/leg_1/motor_2: geometry collision mesh filename=meshes/collision/motor.stl; visual mesh filename=meshes/visual/motor.stl
- link hexapod/leg_2/link_0: geometry collision mesh filename=meshes/collision/leg_0_left.stl; visual mesh filename=meshes/visual/leg_0_left.stl
- link hexapod/leg_2/link_1: geometry collision mesh filename=meshes/collision/leg_1.stl; visual mesh filename=meshes/visual/leg_1.stl
- link hexapod/leg_2/link_2: geometry collision mesh filename=meshes/collision/leg_2_left.stl; visual mesh filename=meshes/visual/leg_2_left.stl
- link hexapod/leg_2/motor_0: geometry collision mesh filename=meshes/collision/motor.stl; visual mesh filename=meshes/visual/motor.stl
- link hexapod/leg_2/motor_1: geometry collision mesh filename=meshes/collision/motor.stl; visual mesh filename=meshes/visual/motor.stl
- link hexapod/leg_2/motor_2: geometry collision mesh filename=meshes/collision/motor.stl; visual mesh filename=meshes/visual/motor.stl
- link hexapod/leg_3/link_0: geometry collision mesh filename=meshes/collision/leg_0_right.stl; visual mesh filename=meshes/visual/leg_0_right.stl
- link hexapod/leg_3/link_1: geometry collision mesh filename=meshes/collision/leg_1.stl; visual mesh filename=meshes/visual/leg_1.stl
- link hexapod/leg_3/link_2: geometry collision mesh filename=meshes/collision/leg_2_right.stl; visual mesh filename=meshes/visual/leg_2_right.stl
- link hexapod/leg_3/motor_0: geometry collision mesh filename=meshes/collision/motor.stl; visual mesh filename=meshes/visual/motor.stl
- link hexapod/leg_3/motor_1: geometry collision mesh filename=meshes/collision/motor.stl; visual mesh filename=meshes/visual/motor.stl
- link hexapod/leg_3/motor_2: geometry collision mesh filename=meshes/collision/motor.stl; visual mesh filename=meshes/visual/motor.stl
- link hexapod/leg_4/link_0: geometry collision mesh filename=meshes/collision/leg_0_left.stl; visual mesh filename=meshes/visual/leg_0_left.stl
- link hexapod/leg_4/link_1: geometry collision mesh filename=meshes/collision/leg_1.stl; visual mesh filename=meshes/visual/leg_1.stl
- link hexapod/leg_4/link_2: geometry collision mesh filename=meshes/collision/leg_2_left.stl; visual mesh filename=meshes/visual/leg_2_left.stl
- link hexapod/leg_4/motor_0: geometry collision mesh filename=meshes/collision/motor.stl; visual mesh filename=meshes/visual/motor.stl
- link hexapod/leg_4/motor_1: geometry collision mesh filename=meshes/collision/motor.stl; visual mesh filename=meshes/visual/motor.stl
- link hexapod/leg_4/motor_2: geometry collision mesh filename=meshes/collision/motor.stl; visual mesh filename=meshes/visual/motor.stl
- link hexapod/leg_5/link_0: geometry collision mesh filename=meshes/collision/leg_0_right.stl; visual mesh filename=meshes/visual/leg_0_right.stl
- link hexapod/leg_5/link_1: geometry collision mesh filename=meshes/collision/leg_1.stl; visual mesh filename=meshes/visual/leg_1.stl
- link hexapod/leg_5/link_2: geometry collision mesh filename=meshes/collision/leg_2_right.stl; visual mesh filename=meshes/visual/leg_2_right.stl
- link hexapod/leg_5/motor_0: geometry collision mesh filename=meshes/collision/motor.stl; visual mesh filename=meshes/visual/motor.stl
- link hexapod/leg_5/motor_1: geometry collision mesh filename=meshes/collision/motor.stl; visual mesh filename=meshes/visual/motor.stl
- link hexapod/leg_5/motor_2: geometry collision mesh filename=meshes/collision/motor.stl; visual mesh filename=meshes/visual/motor.stl

Commit message: Work on the environments
- Added reward function and termination condition to HexapodBullet
- cleanup urdf of hexapod bullet
- Improved init files of environment
- added registration to mujoco and pybullet environments

File: mushroom_rl/environments/pybullet_envs/data/hexapod/hexapod.urdf (robot description, URDF)
Before this commit: robot iiwa, 38 links, 37 joints
Links:
- removed link hexapod/base_link
Joints:
- removed joint hexapod/base_joint

Commit message: Work on hexapod
- minor fixes
- added collision check and penalties

File: mushroom_rl/environments/pybullet_envs/data/hexapod/hexapod.urdf (robot description, URDF)
Before this commit: robot hexapod, 37 links, 36 joints
Joints:
- joint hexapod/leg_0/joint_0: limit lower=-2.356194490192345 upper=2.356194490192345 effort=100 velocity=1.7453292519943295 -> lower=-1.3 upper=1.3 effort=100 velocity=1.7453292519943295
- joint hexapod/leg_1/joint_0: limit lower=-2.356194490192345 upper=2.356194490192345 effort=100 velocity=1.7453292519943295 -> lower=-1.3 upper=1.3 effort=100 velocity=1.7453292519943295
- joint hexapod/leg_2/joint_0: limit lower=-2.356194490192345 upper=2.356194490192345 effort=100 velocity=1.7453292519943295 -> lower=-1.3 upper=1.3 effort=100 velocity=1.7453292519943295
- joint hexapod/leg_3/joint_0: limit lower=-2.356194490192345 upper=2.356194490192345 effort=100 velocity=1.7453292519943295 -> lower=-1.3 upper=1.3 effort=100 velocity=1.7453292519943295
- joint hexapod/leg_4/joint_0: limit lower=-2.356194490192345 upper=2.356194490192345 effort=100 velocity=1.7453292519943295 -> lower=-1.3 upper=1.3 effort=100 velocity=1.7453292519943295
- joint hexapod/leg_5/joint_0: limit lower=-2.356194490192345 upper=2.356194490192345 effort=100 velocity=1.7453292519943295 -> lower=-1.3 upper=1.3 effort=100 velocity=1.7453292519943295
