Commit message: First stub of the manipulator robot

File: mushroom_rl/environments/pybullet_envs/data/manipulator/manipulator.urdf (robot description, URDF)
Before this commit: robot manipulator, 3 links, 2 joints
Links:
- added link manipulator/finger_0_link_0, mass 0.1; collision cylinder length=0.05 radius=0.005; visual cylinder length=0.1 radius=0.005
- added link manipulator/finger_0_link_1, mass 0.1; collision cylinder length=0.1 radius=0.005; visual cylinder length=0.05 radius=0.005
- added link manipulator/finger_1_link_0, mass 0.1; collision cylinder length=0.05 radius=0.005; visual cylinder length=0.1 radius=0.005
- added link manipulator/finger_1_link_1, mass 0.1; collision cylinder length=0.1 radius=0.005; visual cylinder length=0.05 radius=0.005
- added link manipulator/finger_2_link_0, mass 0.1; collision cylinder length=0.05 radius=0.005; visual cylinder length=0.1 radius=0.005
- added link manipulator/finger_2_link_1, mass 0.1; collision cylinder length=0.1 radius=0.005; visual cylinder length=0.05 radius=0.005
- added link manipulator/finger_3_link_0, mass 0.1; collision cylinder length=0.05 radius=0.005; visual cylinder length=0.1 radius=0.005
- added link manipulator/finger_3_link_1, mass 0.1; collision cylinder length=0.1 radius=0.005; visual cylinder length=0.05 radius=0.005
- link manipulator/link_0: geometry collision cylinder length=0.3 radius=0.025; visual cylinder length=0.3 radius=0.025
- link manipulator/link_1: geometry collision cylinder length=0.3 radius=0.025; visual cylinder length=0.3 radius=0.025
Joints:
- added joint manipulator/finger_0_connection: type fixed, parent manipulator/link_0, child manipulator/finger_0_link_0, origin xyz=0 -0.15 0 rpy=0 0 -1.5707963267948966
- added joint manipulator/finger_0_joint: type revolute, parent manipulator/finger_0_link_0, child manipulator/finger_0_link_1, origin xyz=0. 0. -0.1 rpy=0 0 0, axis 0 1 0, limit lower=0 upper=1.5707963267948966 effort=100 velocity=1.0
- added joint manipulator/finger_1_connection: type fixed, parent manipulator/link_0, child manipulator/finger_1_link_0, origin xyz=0 0.15 0 rpy=0 0 1.5707963267948966s
- added joint manipulator/finger_1_joint: type revolute, parent manipulator/finger_1_link_0, child manipulator/finger_1_link_1, origin xyz=0. 0. -0.1 rpy=0 0 0, axis 0 1 0, limit lower=0 upper=1.5707963267948966 effort=100 velocity=1.0
- added joint manipulator/finger_2_connection: type fixed, parent manipulator/link_1, child manipulator/finger_2_link_0, origin xyz=-0.15 0 0 rpy=0 0 -3.141592653589793
- added joint manipulator/finger_2_joint: type revolute, parent manipulator/finger_2_link_0, child manipulator/finger_2_link_1, origin xyz=0. 0. -0.1 rpy=0 0 0, axis 0 1 0, limit lower=0 upper=1.5707963267948966 effort=100 velocity=1.0
- added joint manipulator/finger_3_connection: type fixed, parent manipulator/link_1, child manipulator/finger_3_link_0, origin xyz=0.15 0 0 rpy=0 0 0
- added joint manipulator/finger_3_joint: type revolute, parent manipulator/finger_3_link_0, child manipulator/finger_3_link_1, origin xyz=0. 0. -0.1 rpy=0 0 0, axis 0 1 0, limit lower=0 upper=1.5707963267948966 effort=100 velocity=1.0
- joint manipulator/joint_0: origin xyz=0. 0. 0. rpy=0 1.57079632679 0 -> xyz=0. 0. 0. rpy=0 0 0
- joint manipulator/joint_fixed: origin xyz=0 0 0.25 rpy=1.57079632679 0 0 -> xyz=0 0 0.25 rpy=0 0 0
