Commit message: Fixed joint limit

File: mushroom_rl/environments/pybullet_envs/data/openhand_model_q/model_q.urdf (robot description, URDF)
Before this commit: robot model_q, 14 links, 13 joints
Joints:
- joint base_rot_joint: limit lower=0.0 upper=3.0 effort=10000 velocity=200 -> lower=-0.26179938779 upper=0.26179938779 effort=10000 velocity=200

Commit message: Work on pybullet environments
- Improved Pybullet class to be more flexible
- added concept of simulation state and observation to increase
flexibility of the interface
- Work on OpenHandModelQ
- Added valves
- improved model q urdf
- added joint coupling

File: mushroom_rl/environments/pybullet_envs/data/openhand_model_q/model_q.urdf (robot description, URDF)
Before this commit: robot model_q, 14 links, 13 joints
Links:
- link distal_cl: geometry collision mesh filename=meshes/hand/finger_pp_t_B_round.stl scale=0.00100 0.00100 0.00100; visual mesh filename=meshes/hand/finger_pp_t_B_round.stl scale=0.00100 0.00100 0.00100
- link distal_cr: geometry collision mesh filename=meshes/hand/finger_pp_t_B_round.stl scale=0.00100 0.00100 0.00100; visual mesh filename=meshes/hand/finger_pp_t_B_round.stl scale=0.00100 0.00100 0.00100
- link distal_l: geometry collision mesh filename=meshes/hand/finger_pp_t_B_round.stl scale=0.00100 0.00100 0.00100; visual mesh filename=meshes/hand/finger_pp_t_B_round.stl scale=0.00100 0.00100 0.00100
- link distal_r: geometry collision mesh filename=meshes/hand/finger_pp_t_B_round.stl scale=0.00100 0.00100 0.00100; visual mesh filename=meshes/hand/finger_pp_t_B_round.stl scale=0.00100 0.00100 0.00100
- link prox_cl: geometry collision mesh filename=meshes/hand/proximal.STL scale=0.00100 0.00100 0.00100; visual mesh filename=meshes/hand/proximal.STL scale=0.00100 0.00100 0.00100
- link prox_cr: geometry collision mesh filename=meshes/hand/proximal.STL scale=0.00100 0.00100 0.00100; visual mesh filename=meshes/hand/proximal.STL scale=0.00100 0.00100 0.00100
- link prox_l: geometry collision mesh filename=meshes/hand/proximal.STL scale=0.00100 0.00100 0.00100; visual mesh filename=meshes/hand/proximal.STL scale=0.00100 0.00100 0.00100
- link prox_r: geometry collision mesh filename=meshes/hand/proximal.STL scale=0.00100 0.00100 0.00100; visual mesh filename=meshes/hand/proximal.STL scale=0.00100 0.00100 0.00100
Joints:
- joint fixed1: origin xyz=0. 0.000000 0.01081 rpy=0 1.57079632679 0 -> xyz=0. 0. 0. rpy=0 1.57079632679 0

Commit message: Fixed limits for model q hand
- using more reasonable values for joint, velocity and effort limits

File: mushroom_rl/environments/pybullet_envs/data/openhand_model_q/model_q.urdf (robot description, URDF)
Before this commit: robot model_q, 14 links, 13 joints
Joints:
- joint base_rot_joint: limit lower=-0.26179938779 upper=0.26179938779 effort=10000 velocity=200 -> lower=-0.26179938779 upper=0.26179938779 effort=10 velocity=10
- joint base_to_prox_cl: limit lower=0.0 upper=3.0 effort=10000 velocity=200 -> lower=0.0 upper=2.0 effort=10 velocity=10
- joint base_to_prox_cr: limit lower=0.0 upper=3.0 effort=10000 velocity=200 -> lower=0.0 upper=2.0 effort=10 velocity=10
- joint base_to_prox_l: limit lower=0.0 upper=3.0 effort=10000 velocity=200 -> lower=0.0 upper=2.0 effort=10 velocity=10
- joint base_to_prox_r: limit lower=0.0 upper=3.0 effort=10000 velocity=200 -> lower=0.0 upper=2.0 effort=10 velocity=10
- joint prox_to_distal_cl: limit lower=0.0 upper=1.24 effort=10000 velocity=200 -> lower=0.0 upper=1.24 effort=10 velocity=10
- joint prox_to_distal_cr: limit lower=0.0 upper=1.24 effort=10000 velocity=200 -> lower=0.0 upper=1.24 effort=10 velocity=10
- joint prox_to_distal_l: limit lower=0.0 upper=1.24 effort=10000 velocity=200 -> lower=0.0 upper=1.24 effort=10 velocity=10
- joint prox_to_distal_r: limit lower=0.0 upper=1.24 effort=10000 velocity=200 -> lower=0.0 upper=1.24 effort=10 velocity=10

Commit message: Stl files renamed to lower case

File: mushroom_rl/environments/pybullet_envs/data/openhand_model_q/model_q.urdf (robot description, URDF)
Before this commit: robot model_q, 14 links, 13 joints
Links:
- link prox_cl: geometry collision mesh filename=meshes/hand/proximal.stl scale=0.00100 0.00100 0.00100; visual mesh filename=meshes/hand/proximal.stl scale=0.00100 0.00100 0.00100
- link prox_cr: geometry collision mesh filename=meshes/hand/proximal.stl scale=0.00100 0.00100 0.00100; visual mesh filename=meshes/hand/proximal.stl scale=0.00100 0.00100 0.00100
- link prox_l: geometry collision mesh filename=meshes/hand/proximal.stl scale=0.00100 0.00100 0.00100; visual mesh filename=meshes/hand/proximal.stl scale=0.00100 0.00100 0.00100
- link prox_r: geometry collision mesh filename=meshes/hand/proximal.stl scale=0.00100 0.00100 0.00100; visual mesh filename=meshes/hand/proximal.stl scale=0.00100 0.00100 0.00100

Commit message: Work on model_q urdf
- scaled down finger meshes
- fixed copy-paste error in collision meshes
- now hand looks reasonable

File: mushroom_rl/environments/pybullet_envs/data/openhand_model_q/model_q.urdf (robot description, URDF)
Before this commit: robot model_q, 14 links, 13 joints
Links:
- link distal_cl: geometry collision mesh filename=meshes/hand/finger_pp_t_B_round.stl; visual mesh filename=meshes/hand/finger_pp_t_B_round.stl
- link distal_cr: geometry collision mesh filename=meshes/hand/finger_pp_t_B_round.stl; visual mesh filename=meshes/hand/finger_pp_t_B_round.stl
- link distal_l: geometry collision mesh filename=meshes/hand/finger_pp_t_B_round.stl; visual mesh filename=meshes/hand/finger_pp_t_B_round.stl
- link distal_r: geometry collision mesh filename=meshes/hand/finger_pp_t_B_round.stl; visual mesh filename=meshes/hand/finger_pp_t_B_round.stl
- link prox_cl: geometry collision mesh filename=meshes/hand/proximal.stl; visual mesh filename=meshes/hand/proximal.stl
- link prox_cr: geometry collision mesh filename=meshes/hand/proximal.stl; visual mesh filename=meshes/hand/proximal.stl
- link prox_l: geometry collision mesh filename=meshes/hand/proximal.stl; visual mesh filename=meshes/hand/proximal.stl
- link prox_r: geometry collision mesh filename=meshes/hand/proximal.stl; visual mesh filename=meshes/hand/proximal.stl

Commit message: leanup of mesh files in openhand model q

File: mushroom_rl/environments/pybullet_envs/data/openhand_model_q/model_q.urdf (robot description, URDF)
Before this commit: robot model_q, 14 links, 13 joints
Links:
- link distal_cl: geometry collision mesh filename=meshes/hand/distal.stl; visual mesh filename=meshes/hand/distal.stl
- link distal_cr: geometry collision mesh filename=meshes/hand/distal.stl; visual mesh filename=meshes/hand/distal.stl
- link distal_l: geometry collision mesh filename=meshes/hand/distal.stl; visual mesh filename=meshes/hand/distal.stl
- link distal_r: geometry collision mesh filename=meshes/hand/distal.stl; visual mesh filename=meshes/hand/distal.stl

Commit message: Minor fixes for Model Q environment and URDF

File: mushroom_rl/environments/pybullet_envs/data/openhand_model_q/model_q.urdf (robot description, URDF)
Before this commit: robot model_q, 14 links, 13 joints
Links:
- link distal_cl: mass 0.1 -> 0.015
- link distal_cr: mass 0.1 -> 0.015
- link distal_l: mass 0.1 -> 0.015
- link distal_r: mass 0.1 -> 0.015
- link prox_cl: mass 0.1 -> 0.03
- link prox_cr: mass 0.1 -> 0.03
- link prox_l: mass 0.1 -> 0.03
- link prox_r: mass 0.1 -> 0.03
Joints:
- joint base_rot_joint: limit lower=-0.26179938779 upper=0.26179938779 effort=10 velocity=10 -> lower=-0.26179938779 upper=0.26179938779 effort=10 velocity=50
- joint base_to_prox_cl: limit lower=0.0 upper=2.0 effort=10 velocity=10 -> lower=0.0 upper=2.0 effort=10 velocity=50
- joint base_to_prox_cr: limit lower=0.0 upper=2.0 effort=10 velocity=10 -> lower=0.0 upper=2.0 effort=10 velocity=50
- joint base_to_prox_l: limit lower=0.0 upper=2.0 effort=10 velocity=10 -> lower=0.0 upper=2.0 effort=10 velocity=50
- joint base_to_prox_r: limit lower=0.0 upper=2.0 effort=10 velocity=10 -> lower=0.0 upper=2.0 effort=10 velocity=50
- joint prox_to_distal_cl: limit lower=0.0 upper=1.24 effort=10 velocity=10 -> lower=0.0 upper=1.24 effort=10 velocity=50
- joint prox_to_distal_cr: limit lower=0.0 upper=1.24 effort=10 velocity=10 -> lower=0.0 upper=1.24 effort=10 velocity=50
- joint prox_to_distal_l: limit lower=0.0 upper=1.24 effort=10 velocity=10 -> lower=0.0 upper=1.24 effort=10 velocity=50
- joint prox_to_distal_r: limit lower=0.0 upper=1.24 effort=10 velocity=10 -> lower=0.0 upper=1.24 effort=10 velocity=50
