Commit message: Change the maximum effort of the joint

File: mushroom_rl/environments/pybullet_envs/data/air_hockey/planar/planar_robot_1.urdf (robot description, URDF)
Before this commit: robot planar_robot_1, 7 links, 6 joints
Joints:
- joint planar_robot_1/joint_1: limit lower=-2.9670597283903604 upper=2.9670597283903604 effort=320.0 velocity=2.35619449019 -> lower=-2.9670597283903604 upper=2.9670597283903604 effort=40.0 velocity=2.35619449019
- joint planar_robot_1/joint_2: limit lower=-2.0943951023931953 upper=2.0943951023931953 effort=320.0 velocity=2.35619449019 -> lower=-2.0943951023931953 upper=2.0943951023931953 effort=30.0 velocity=2.35619449019
- joint planar_robot_1/joint_3: limit lower=-2.0943951023931953 upper=2.0943951023931953 effort=320.0 velocity=2.35619449019 -> lower=-2.0943951023931953 upper=2.0943951023931953 effort=20.0 velocity=2.35619449019

File: mushroom_rl/environments/pybullet_envs/data/air_hockey/planar/planar_robot_2.urdf (robot description, URDF)
Before this commit: robot planar_robot_2, 7 links, 6 joints
Joints:
- joint planar_robot_2/joint_1: limit lower=-2.9670597283903604 upper=2.9670597283903604 effort=320.0 velocity=2.35619449019 -> lower=-2.9670597283903604 upper=2.9670597283903604 effort=40.0 velocity=2.35619449019
- joint planar_robot_2/joint_2: limit lower=-2.0943951023931953 upper=2.0943951023931953 effort=320.0 velocity=2.35619449019 -> lower=-2.0943951023931953 upper=2.0943951023931953 effort=30.0 velocity=2.35619449019
- joint planar_robot_2/joint_3: limit lower=-2.0943951023931953 upper=2.0943951023931953 effort=320.0 velocity=2.35619449019 -> lower=-2.0943951023931953 upper=2.0943951023931953 effort=20.0 velocity=2.35619449019

Commit message: Change the inertial of planar robot
- Add state normalization for the air_hockey_env
- Use more realistic inertia

File: mushroom_rl/environments/pybullet_envs/data/air_hockey/planar/planar_robot_1.urdf (robot description, URDF)
Before this commit: robot planar_robot_1, 7 links, 6 joints
Links:
- link planar_robot_1/link_1: mass 1 -> 3
- link planar_robot_1/link_2: mass 1 -> 2.4
- link planar_robot_1/link_3: mass 1 -> 2.4
Joints:
- joint planar_robot_1/joint_2: limit lower=-2.0943951023931953 upper=2.0943951023931953 effort=30.0 velocity=2.35619449019 -> lower=-2.0943951023931953 upper=2.0943951023931953 effort=15.0 velocity=2.35619449019
- joint planar_robot_1/joint_3: limit lower=-2.0943951023931953 upper=2.0943951023931953 effort=20.0 velocity=2.35619449019 -> lower=-2.0943951023931953 upper=2.0943951023931953 effort=2.0 velocity=2.35619449019

File: mushroom_rl/environments/pybullet_envs/data/air_hockey/planar/planar_robot_2.urdf (robot description, URDF)
Before this commit: robot planar_robot_2, 7 links, 6 joints
Links:
- link planar_robot_2/link_1: mass 1 -> 3
- link planar_robot_2/link_2: mass 1 -> 2.4
- link planar_robot_2/link_3: mass 1 -> 2.4
Joints:
- joint planar_robot_2/joint_2: limit lower=-2.0943951023931953 upper=2.0943951023931953 effort=30.0 velocity=2.35619449019 -> lower=-2.0943951023931953 upper=2.0943951023931953 effort=15.0 velocity=2.35619449019
- joint planar_robot_2/joint_3: limit lower=-2.0943951023931953 upper=2.0943951023931953 effort=20.0 velocity=2.35619449019 -> lower=-2.0943951023931953 upper=2.0943951023931953 effort=2.0 velocity=2.35619449019
