Commit message: Change the collision model of puck

File: mushroom_rl/environments/pybullet_envs/data/air_hockey/puck.urdf (robot description, URDF)
Before this commit: robot puck, 1 links, 0 joints
Links:
- link Puck_link: geometry collision cylinder length=0.02 radius=0.03165; visual cylinder length=0.0049 radius=0.03165

Commit message: Reset the collision model of the puck

File: mushroom_rl/environments/pybullet_envs/data/air_hockey/puck.urdf (robot description, URDF)
Before this commit: robot puck, 1 links, 0 joints
Links:
- link Puck_link: geometry collision cylinder length=0.0049 radius=0.03165; visual cylinder length=0.0049 radius=0.03165
